Commit message: Correct hokuyo.dae path

File: turtlebot_udg_description/urdf/sensors/hokuyo.urdf.xacro (robot description, xacro)
@@ -20,5 +20,5 @@
 		<origin xyz="0 0 0" rpy="0 0 0"/>
 		<geometry>
-		  <mesh filename="package://turtlebot_description/meshes/sensors/hokuyo.dae"/>
+		  <mesh filename="package://turtlebot_udg_description/meshes/sensors/hokuyo.dae"/>
 		</geometry>
 	      </visual>

Commit message: Modified and deleted some comments

File: turtlebot_udg_description/urdf/sensors/hokuyo.urdf.xacro (robot description, xacro)
@@ -5,5 +5,4 @@
 	<xacro:macro name="sensor_hokuyo" params="parent">
 	    <joint name="hokuyo_joint" type="fixed">
-	      <!--<axis xyz="0 1 0" />-->
 	      <origin xyz="0.075 0 0.225" rpy="0 0 0"/>
 	      <parent link="${parent}"/>

File: turtlebot_udg_description/urdf/turtlebot_udg_gazebo.urdf.xacro (robot description, xacro)
@@ -1,5 +1,5 @@
 <?xml version="1.0"?>
 <robot name="turtlebot_udg_gazebo" xmlns:xacro="http://ros.org/wiki/xacro">
-  <!-- Microsoft Kinect / ASUS Xtion PRO Live for simulation -->
+  <!-- Hokuyo sensor for simulation -->
   <xacro:macro name="turtlebot_sim_laser_range_finder">
    <gazebo reference="hokuyo_link">

Commit message: Inertial matrix changed

File: turtlebot_udg_description/urdf/sensors/hokuyo.urdf.xacro (robot description, xacro)
@@ -25,5 +25,5 @@
 		<mass value="0.16" />
      		<origin xyz="0 0 0" rpy="0 0 0"/>
-      		<inertia ixx="1e-6" ixy="0" ixz="0" iyy="1e-6" iyz="0" izz="1e-6" />
+      		<inertia ixx="9.866e-5" ixy="0" ixz="0" iyy="6.667e-5" iyz="0" izz="9.866e-5" />
 	      </inertial>
 	    </link>

Commit message: Changed hokuyo posicion

File: turtlebot_udg_description/urdf/sensors/hokuyo.urdf.xacro (robot description, xacro)
@@ -5,5 +5,5 @@
 	<xacro:macro name="sensor_hokuyo" params="parent">
 	    <joint name="hokuyo_joint" type="fixed">
-	      <origin xyz="0.075 0 0.225" rpy="0 0 0"/>
+	      <origin xyz="0.075 0 0.43" rpy="0 0 0"/>
 	      <parent link="${parent}"/>
 	      <child link="hokuyo_link"/>
