Commit message: Kinect sensor added

File: turtlebot_udg_description/robots/kobuki_hexagons_hokuyo.urdf.xacro (robot description, xacro)
@@ -3,5 +3,5 @@
     - Base      : kobuki
     - Stacks    : hexagons
-    - 3d Sensor : hokuyo
+    - 3d Sensor : kinect and hokuyo
 -->
 <robot name="turtlebot" xmlns:xacro="http://ros.org/wiki/xacro">
@@ -9,7 +9,9 @@
   <xacro:include filename="$(find kobuki_description)/urdf/kobuki.urdf.xacro" />
   <xacro:include filename="$(find turtlebot_description)/urdf/stacks/hexagons.urdf.xacro"/>
+  <xacro:include filename="$(find turtlebot_description)/urdf/sensors/kinect.urdf.xacro"/>
   <xacro:include filename="$(find turtlebot_udg_description)/urdf/sensors/hokuyo.urdf.xacro"/>
   <xacro:kobuki/>
   <xacro:stack_hexagons parent="base_link"/>
+  <xacro:sensor_kinect parent="base_link"/>
   <xacro:sensor_hokuyo parent="base_link"/>
 </robot>

File: turtlebot_udg_description/urdf/turtlebot_udg_gazebo.urdf.xacro (robot description, xacro)
@@ -2,45 +2,7 @@
 <robot name="turtlebot_udg_gazebo" xmlns:xacro="http://ros.org/wiki/xacro">
   <!-- Microsoft Kinect / ASUS Xtion PRO Live for simulation -->
-  <xacro:macro name="turtlebot_sim_3dsensor">
-    <gazebo reference="camera_link">
-      <sensor type="depth" name="camera">
-        <always_on>true</always_on>
-        <update_rate>20.0</update_rate>
-        <camera>
-          <horizontal_fov>${60.0*M_PI/180.0}</horizontal_fov>
-          <image>
-            <format>B8G8R8</format>
-            <width>640</width>
-            <height>480</height>
-          </image>
-          <clip>
-            <near>0.05</near>
-            <far>8.0</far>
-          </clip>
-        </camera>
-        <plugin name="kinect_camera_controller" filename="libgazebo_ros_openni_kinect.so">
-          <cameraName>camera</cameraName>
-          <alwaysOn>true</alwaysOn>
-          <updateRate>10</updateRate>
-          <imageTopicName>rgb/image_raw</imageTopicName>
-          <depthImageTopicName>depth/image_raw</depthImageTopicName>
-          <pointCloudTopicName>depth/points</pointCloudTopicName>
-          <cameraInfoTopicName>rgb/camera_info</cameraInfoTopicName>
-          <depthImageCameraInfoTopicName>depth/camera_info</depthImageCameraInfoTopicName>
-          <frameName>camera_depth_optical_frame</frameName>
-          <baseline>0.1</baseline>
-          <distortion_k1>0.0</distortion_k1>
-          <distortion_k2>0.0</distortion_k2>
-          <distortion_k3>0.0</distortion_k3>
-          <distortion_t1>0.0</distortion_t1>
-          <distortion_t2>0.0</distortion_t2>
-          <pointCloudCutoff>0.4</pointCloudCutoff>
-        </plugin>
-      </sensor>
-    </gazebo>
-  </xacro:macro>
   <xacro:macro name="turtlebot_sim_laser_range_finder">
    <gazebo reference="hokuyo_link">
-      <sensor type="gpu_ray" name="head_hokuyo_sensor">
+      <sensor type="ray" name="head_hokuyo_sensor">
         <pose>0 0 0 0 0 0</pose>
         <visualize>true</visualize>
@@ -66,5 +28,5 @@
           </noise>
         </ray>
-        <plugin name="gazebo_ros_head_hokuyo_controller" filename="libgazebo_ros_gpu_laser.so">
+        <plugin name="gazebo_ros_head_hokuyo_controller" filename="libgazebo_ros_laser.so">
           <topicName>/hokuyo_scan</topicName>
           <frameName>hokuyo_link</frameName>

Commit message: Parameters added in launch file

File: turtlebot_udg_description/robots/kobuki_hexagons_hokuyo.urdf.xacro (robot description, xacro)
@@ -14,4 +14,4 @@
   <xacro:stack_hexagons parent="base_link"/>
   <xacro:sensor_kinect parent="base_link"/>
-  <xacro:sensor_hokuyo parent="base_link"/>
+  <xacro:sensor_hokuyo parent="base_link" visual="$(arg visual)" stddev="$(arg stddev)"/>
 </robot>

File: turtlebot_udg_description/urdf/sensors/hokuyo.urdf.xacro (robot description, xacro)
@@ -3,5 +3,5 @@
   <xacro:include filename="$(find turtlebot_udg_description)/urdf/turtlebot_udg_gazebo.urdf.xacro"/>
   <xacro:include filename="$(find turtlebot_description)/urdf/turtlebot_properties.urdf.xacro"/>
-	<xacro:macro name="sensor_hokuyo" params="parent">
+	<xacro:macro name="sensor_hokuyo" params="parent visual stddev">
 	    <joint name="hokuyo_joint" type="fixed">
 	      <origin xyz="0.075 0 0.43" rpy="0 0 0"/>
@@ -29,5 +29,5 @@
 	    </link>
 	     <!-- Hokuyo sensor for simulation -->
-	     <xacro:turtlebot_sim_laser_range_finder/>
+	     <xacro:turtlebot_sim_laser_range_finder visual="$(arg visual)" stddev="$(arg stddev)"/>
 	</xacro:macro>
 </robot>

File: turtlebot_udg_description/urdf/turtlebot_udg_gazebo.urdf.xacro (robot description, xacro)
@@ -2,9 +2,9 @@
 <robot name="turtlebot_udg_gazebo" xmlns:xacro="http://ros.org/wiki/xacro">
   <!-- Hokuyo sensor for simulation -->
-  <xacro:macro name="turtlebot_sim_laser_range_finder">
+  <xacro:macro name="turtlebot_sim_laser_range_finder" params="visual stddev">
    <gazebo reference="hokuyo_link">
       <sensor type="ray" name="head_hokuyo_sensor">
         <pose>0 0 0 0 0 0</pose>
-        <visualize>true</visualize>
+        <visualize>${visual}</visualize>
         <update_rate>40</update_rate>
         <ray>
@@ -25,5 +25,5 @@
             <type>gaussian</type>
             <mean>0.0</mean>
-            <stddev>0.01</stddev>
+            <stddev>${stddev}</stddev>
           </noise>
         </ray>
